File: Hardware/SparkFun_Ardumoto.sch (EAGLE design)
At the start: 66 parts, among them U1 ARDUINO, U2 L298, U5 74HC1G04, U6 74HC1G04

Commit message: Made post-review changes
Other:
- note added: "The following jumpers are used to set the ArduMoto's control pins to one of two possible connection points. Leave jumpers completely open if manually connecting control lines. The default PWM pins are assigned to arduino timer 2, while the alternate assigns them to timer 1. JP1: 'A' Direction -- set to D2 (default) or D8 JP2: 'A' PWM signal -- set to D3 (default) or D9 JP3: 'B' Direction -- set t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"
- note removed: "The folloing jumpers are used to set the ArduMoto's control pins to one of two possible connection points. Leave jumpers completely open if manually connecting control lines. JP1: 'A' Direction -- set to D8 (default) or D3 JP2: 'A' PWM signal -- set to D9 (default) or D5 JP3: 'B' Direction -- set to D7 (default) or D2 JP4: 'B' PWM signal -- set to D10 (default) or D6"
Changed lines of the file:
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@@
 <text x="238.76" y="7.62" size="2.54" layer="94" font="vector">v20</text>
 <text x="168.148" y="8.636" size="2.54" layer="94" font="vector" align="center-left">Revised by: Marshall Taylor</text>
-<text x="152.4" y="172.72" size="2.032" layer="97" font="vector" align="top-left">The folloing jumpers are used to set the ArduMoto's
+<text x="152.4" y="172.72" size="2.032" layer="97" font="vector" align="top-left">The following jumpers are used to set the ArduMoto's
   control pins to one of two possible connection
   points.
 Leave jumpers completely open if manually connecting
   control lines.
-JP1: 'A' Direction -- set to D8 (default) or D3
-JP2: 'A' PWM signal -- set to D9 (default) or D5
-JP3: 'B' Direction -- set to D7 (default) or D2
-JP4: 'B' PWM signal -- set to D10 (default) or D6</text>
+The default PWM pins are assigned to arduino
+timer 2, while the alternate assigns them to timer 1.
+JP1: 'A' Direction -- set to D2 (default) or D8
+JP2: 'A' PWM signal -- set to D3 (default) or D9
+JP3: 'B' Direction -- set to D4 (default) or D7
+JP4: 'B' PWM signal -- set to D11 (default) or D10</text>
 <text x="5.08" y="177.8" size="3.175" layer="97" font="vector">Power Circuits</text>
 <text x="168.148" y="11.176" size="2.54" layer="94" font="vector">Pete Dokter</text>

Commit message: switched components LED1 and LED3
Parts:
- LED1: value Yellow -> BLUE; device SparkFun-LED:LED-YELLOW0603 -> SparkFun-LED:LED-BLUE0603
- LED3: value BLUE -> Yellow; device SparkFun-LED:LED-BLUE0603 -> SparkFun-LED:LED-YELLOW0603
Changed lines of the file:
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@@
 <part name="R3" library="SparkFun-Resistors" deviceset="1KOHM" device="-0603-1/10W-1%" value="1k"/>
 <part name="R4" library="SparkFun-Resistors" deviceset="1KOHM" device="-0603-1/10W-1%" value="1k"/>
-<part name="LED1" library="SparkFun-LED" deviceset="LED-YELLOW" device="0603" value="Yellow"/>
-<part name="LED3" library="SparkFun-LED" deviceset="LED-BLUE" device="0603" value="BLUE"/>
+<part name="LED1" library="SparkFun-LED" deviceset="LED-BLUE" device="0603" value="BLUE"/>
+<part name="LED3" library="SparkFun-LED" deviceset="LED-YELLOW" device="0603" value="Yellow"/>
 <part name="D1" library="SparkFun-DiscreteSemi" deviceset="DIODE-SCHOTTKY" device="-SS14" value="1A/40V/500mV"/>
 <part name="D2" library="SparkFun-DiscreteSemi" deviceset="DIODE-SCHOTTKY" device="-SS14" value="1A/40V/500mV"/>
